File: hardware/NERD-HPC/NERD-HPC.kicad_pcb (KiCad board)
At the start: 4 copper layers, 137 x 72 mm, 157 parts, among them J1 USB_C_Receptacle, J2 Micro_SD_Card_Det_Hirose_DM3AT, J3 Conn_01x06_Socket, J4 Conn_01x06_Socket, Q1 Q_PMOS_GSD, Q2 Q_NMOS_GSD, SW1 SW_Push, SW10 SW_Push, SW11 SW_Push, SW12 SW_Push, SW13 SW_Push, SW14 SW_Push, SW15 SW_Push, SW16 SW_Push, SW17 SW_Push, SW18 SW_Push, SW19 SW_Push, SW2 SW_Push, SW20 SW_Push, SW21 SW_Push, SW22 SW_Push, SW23 SW_Push, SW24 SW_Push, SW25 SW_Push, SW26 SW_Push, SW27 SW_Push, SW28 SW_Push, SW29 SW_Push, SW3 SW_SPDT_312, SW30 SW_Push, SW31 SW_Push, SW32 SW_Push, SW33 SW_Push, SW34 SW_Push, SW35 SW_Push, SW36 SW_Push, SW37 SW_Push, SW38 SW_Push, SW39 SW_Push, SW4 SW_SPDT_312, SW40 SW_Push, SW41 SW_Push, SW42 SW_Push, SW43 SW_Push, SW44 SW_Push, SW45 SW_Push, SW46 SW_Push, SW47 SW_Push, SW48 SW_Push, SW49 SW_Push, SW5 SW_SPDT_312, SW50 SW_Push, SW51 SW_Push, SW52 SW_Push, SW53 SW_Push, SW54 SW_Push, SW55 SW_Push, SW56 SW_Push, SW57 SW_Push, SW58 SW_Push, SW59 SW_Push, SW6 SW_Push, SW60 SW_Push, SW61 SW_Push, SW62 SW_Push, SW63 SW_Push, SW64 SW_Push, SW65 SW_Push, SW66 SW_Push, SW67 SW_Push, SW68 SW_Push, SW69 SW_Push, SW7 SW_Push, SW70 SW_Push, SW8 SW_Push, SW9 SW_Push, U1 RP2040, U2 NJM2845DL1-33, U3 W25Q32JVSS, U4 MCP23017_SP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

Commit message: NERD HPC pcb Rev.4
Other:
- board text added: "Rev.4"
- board text removed: "Rev.3"
Changed lines of the file:
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@@
 		(tags "switch single-pole opposite-side-connection double-throw SPDT würth wurth")
 		(property "Reference" "SW4"
-			(at 0 2.576102 90)
+			(at 4.953 0 180)
 			(layer "F.SilkS")
 			(effects
@@
 		(at 139.173949 87.708)
 		(property "Reference" "RV2"
-			(at -3.436349 -2.364 0)
+			(at 0.018051 -3.761 0)
 			(unlocked yes)
 			(layer "F.SilkS")
@@
 		(tags "capacitor")
 		(property "Reference" "C17"
-			(at -1.905 0.722 0)
+			(at -1.905 0.087 0)
 			(layer "B.SilkS")
 			(effects
@@
 		(tags "resistor")
 		(property "Reference" "R17"
-			(at 0.317 -3.377 180)
+			(at -0.064 1.195 180)
 			(layer "B.SilkS")
 			(effects
@@
 		(tags "resistor")
 		(property "Reference" "R15"
-			(at 0 -3.377 0)
+			(at 0 1.195 0)
 			(layer "B.SilkS")
 			(effects
@@
 		(tags "resistor")
 		(property "Reference" "R2"
-			(at 4.826 0 90)
+			(at 2.159 0 90)
 			(layer "B.SilkS")
 			(effects
@@
 		(tags "capacitor")
 		(property "Reference" "C9"
-			(at 2.286 -1.016 180)
+			(at 1.778 0 90)
 			(layer "B.SilkS")
 			(effects
@@
 		(tags "capacitor")
 		(property "Reference" "C16"
-			(at 0.254 1.528 90)
+			(at -0.127 1.31 90)
 			(layer "B.SilkS")
 			(effects
@@
 		(tags "DPAK TO-252 DPAK-3 TO-252-3 SOT-428")
 		(property "Reference" "U2"
-			(at 0 4.5 0)
+			(at 0.049 -4.3055 0)
 			(layer "B.SilkS")
 			(effects
@@
 		(tags "SOT TO_SOT_SMD")
 		(property "Reference" "Q1"
-			(at -0.762 0 0)
+			(at 1.9835 1.077 180)
 			(layer "B.SilkS")
 			(effects
@@
 		(tags "resistor")
 		(property "Reference" "R16"
-			(at 0 -3.377 0)
+			(at 0 1.195 0)
 			(layer "B.SilkS")
 			(effects
@@
 		(tags "capacitor")
 		(property "Reference" "C15"
-			(at 0 -1.27 0)
+			(at 2.794 0 0)
 			(layer "B.SilkS")
 			(effects
@@
 		(tags "capacitor")
 		(property "Reference" "C2"
-			(at 2.032 0 90)
+			(at 2.032 0.254 90)
 			(layer "B.SilkS")
 			(effects
@@
 		(tags "resistor")
 		(property "Reference" "R14"
-			(at 0 3.377 0)
+			(at 0 -1.195 0)
 			(layer "B.SilkS")
 			(effects
@@
 		(layer "Edge.Cuts")
 	)
-	(gr_text "Rev.3"
+	(gr_text "Rev.4"
 		(at 215 142 0)
 		(layer "B.SilkS")
