File: hardware/NERD-HPC_CASE_F/NERD-HPC_CASE_F.kicad_pcb (KiCad board)
At the start: 2 copper layers, 137 x 72 mm, 71 parts

Commit message: NERD HPC CASE F pcb Rev.4
Other:
- board text added: "IO3"
- board text added: "IO4"
- board text added: "Rev.4"
- board text added: "hello, nerld"
- board text removed: "IO3_A"
- board text removed: "IO4_A"
- board text removed: "Rev.3"
Changed lines of the file:
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@@
 		(layer "Edge.Cuts")
 	)
-	(gr_text "Rev.3"
+	(gr_text "hello, nerld"
+		(at 97 83.8 0)
+		(layer "B.SilkS")
+		(effects
+			(font
+				(size 1 1)
+				(thickness 0.1)
+			)
+			(justify bottom mirror)
+		)
+	)
+	(gr_text "Rev.4"
 		(at 195.5 130 0)
 		(layer "B.SilkS")
@@
 		)
 	)
-	(gr_text "IO3_A"
+	(gr_text "IO3"
 		(at 195.122 63.708 90)
 		(layer "F.SilkS")
@@
 		)
 	)
-	(gr_text "IO4_A"
+	(gr_text "IO4"
 		(at 197.662 63.708 90)
 		(layer "F.SilkS")
